Commit message: Imported upstream version '1.0.0' of 'upstream'

File: turtlebot4_description/urdf/lite/turtlebot4.urdf.xacro (robot description, xacro)
@@ -21,8 +21,8 @@
             rpy="0 0 ${pi/2}"/>
   </xacro:rplidar>
-  <xacro:camera_bracket name="oakd_lite_camera_bracket" parent_link="base_link">
+  <xacro:camera_bracket name="oakd_camera_bracket" parent_link="base_link">
     <origin xyz="${camera_mount_x_offset} ${camera_mount_y_offset} ${camera_mount_z_offset + base_link_z_offset}"/>
   </xacro:camera_bracket>
-  <xacro:oakd name="oakd_lite" parent_link="oakd_lite_camera_bracket">
+  <xacro:oakd model="lite" parent_link="oakd_camera_bracket">
     <origin xyz="${oakd_lite_x_offset} ${oakd_lite_y_offset} ${oakd_lite_z_offset}"/>
   </xacro:oakd>

File: turtlebot4_description/urdf/sensors/oakd.urdf.xacro (robot description, xacro)
@@ -1,5 +1,5 @@
 <?xml version="1.0"?>
 <robot xmlns:xacro="http://ros.org/wiki/xacro">
-<xacro:macro name="oakd" params="name parent_link *origin">
+<xacro:macro name="oakd" params="name:=oakd parent_link *origin model:=pro">
   <xacro:include filename="$(find irobot_create_description)/urdf/common_properties.urdf.xacro"/>
   <xacro:property name="mass"       value="0.061"/>
@@ -22,5 +22,5 @@
     <visual>
       <geometry>
-        <mesh filename="package://turtlebot4_description/meshes/${name}.dae" scale="1 1 1" />
+        <mesh filename="package://turtlebot4_description/meshes/${name}_${model}.dae" scale="1 1 1" />
       </geometry>
     </visual>

File: turtlebot4_description/urdf/standard/turtlebot4.urdf.xacro (robot description, xacro)
@@ -95,8 +95,8 @@
             rpy="0 0 ${pi/2}"/>
   </xacro:rplidar>
-  <xacro:camera_bracket name="oakd_pro_camera_bracket">
+  <xacro:camera_bracket name="oakd_camera_bracket">
     <origin xyz="${camera_mount_x_offset} ${camera_mount_y_offset} ${camera_mount_z_offset}"/>
   </xacro:camera_bracket>
-  <xacro:oakd name="oakd_pro" parent_link="oakd_pro_camera_bracket">
+  <xacro:oakd model="pro" parent_link="oakd_camera_bracket">
     <origin xyz="${oakd_pro_x_offset} ${oakd_pro_y_offset} ${oakd_pro_z_offset}"/>
   </xacro:oakd>
